Commit message: added mapper params

File: description/robot_core.xacro (robot description, xacro)
@@ -16,4 +16,12 @@
     <!-- BASE LINK -->
     <link name="base_link">
+    </link>
+    <!-- <Base Footprint Link> -->
+    <joint name="base_footprint_link" type="fixed">
+        <parent link="base_link"/>
+        <child link="base_footprint"/>
+        <origin xyz="0.0 0.0 0.0" rpy="0.0 0.0 0.0"/>
+    </joint>
+    <link name="base_footprint">
     </link>
     <!-- CHASSIS LINK -->
